Commit message: change path convention for newer structure. untested.

File: urdf/gummi_description.urdf (robot description, URDF)
Before this commit: robot gummi, 9 links, 8 joints
Links:
- link base_link: geometry collision mesh filename=package://gummi_base_template/meshes/base_link.STL; visual mesh filename=package://gummi_base_template/meshes/base_link.STL
- link gripper_Link: geometry collision mesh filename=package://gummi_base_template/meshes/gripper_Link.stl
- link lowerarm: geometry collision mesh filename=package://gummi_base_template/meshes/j6_Link.STL; visual mesh filename=package://gummi_base_template/meshes/j6_Link.STL
- link lowerarm_preroll: geometry collision mesh filename=package://gummi_base_template/meshes/j5_Link.STL; visual mesh filename=package://gummi_base_template/meshes/j5_Link.STL
- link shoulder: geometry collision mesh filename=package://gummi_base_template/meshes/j2_Link.STL; visual mesh filename=package://gummi_base_template/meshes/j2_Link.STL
- link shoulder_preroll: geometry collision mesh filename=package://gummi_base_template/meshes/j1_Link.STL; visual mesh filename=package://gummi_base_template/meshes/j1_Link.STL
- link upperarm: geometry collision mesh filename=package://gummi_base_template/meshes/j4_Link.STL; visual mesh filename=package://gummi_base_template/meshes/j4_Link.STL
- link upperarm_preroll: geometry collision mesh filename=package://gummi_base_template/meshes/j3_Link.STL; visual mesh filename=package://gummi_base_template/meshes/j3_Link.STL
- link wrist: geometry collision mesh filename=package://gummi_base_template/meshes/j7_Link.STL; visual mesh filename=package://gummi_base_template/meshes/j7_Link.STL

Commit message: changed the path for the mesh files

File: urdf/gummi_description.urdf (robot description, URDF)
Before this commit: robot gummi, 9 links, 8 joints
Links:
- link base_link: geometry collision mesh filename=package://gummi_base_ghost/meshes/base_link.STL; visual mesh filename=package://gummi_base_ghost/meshes/base_link.STL
- link gripper_Link: geometry collision mesh filename=package://gummi_ee_raspberry/meshes/gripper_Link.stl
- link lowerarm: geometry collision mesh filename=package://gummi_ee_raspberry/meshes/j6_Link.STL; visual mesh filename=package://gummi_ee_raspberry/meshes/j6_Link.STL
- link lowerarm_preroll: geometry collision mesh filename=package://gummi_ee_raspberry/meshes/j5_Link.STL; visual mesh filename=package://gummi_ee_raspberry/meshes/j5_Link.STL
- link shoulder: geometry collision mesh filename=package://gummi_base_ghost/meshes/j2_Link.STL; visual mesh filename=package://gummi_base_ghost/meshes/j2_Link.STL
- link shoulder_preroll: geometry collision mesh filename=package://gummi_base_ghost/meshes/j1_Link.STL; visual mesh filename=package://gummi_base_ghost/meshes/j1_Link.STL
- link upperarm: geometry collision mesh filename=package://gummi_base_ghost/meshes/j4_Link.STL; visual mesh filename=package://gummi_base_ghost/meshes/j4_Link.STL
- link upperarm_preroll: geometry collision mesh filename=package://gummi_base_ghost/meshes/j3_Link.STL; visual mesh filename=package://gummi_base_ghost/meshes/j3_Link.STL
- link wrist: geometry collision mesh filename=package://gummi_ee_raspberry/meshes/j7_Link.STL; visual mesh filename=package://gummi_ee_raspberry/meshes/j7_Link.STL
Joints:
- joint wrist_pitch: axis 0 1 0 -> 0 -1 0

File: xacro/gummi_description_base.urdf.xacro (robot description, xacro)
@@ -23,19 +23,19 @@
       <geometry>
         <mesh
-          filename="package://gummi_base_template/meshes/base_link.STL" />
-      </geometry>
-      <material
-        name="">
-        <color
-          rgba="0.79216 0.81961 0.93333 1" />
-      </material>
-    </visual>
-    <collision>
-      <origin
-        xyz="0 0 0"
-        rpy="0 0 0" />
-      <geometry>
-        <mesh
-          filename="package://gummi_base_template/meshes/base_link.STL" />
+          filename="package://gummi_base_ghost/meshes/base_link.STL" />
+      </geometry>
+      <material
+        name="">
+        <color
+          rgba="0.79216 0.81961 0.93333 1" />
+      </material>
+    </visual>
+    <collision>
+      <origin
+        xyz="0 0 0"
+        rpy="0 0 0" />
+      <geometry>
+        <mesh
+          filename="package://gummi_base_ghost/meshes/base_link.STL" />
       </geometry>
     </collision>
@@ -64,19 +64,19 @@
       <geometry>
         <mesh
-          filename="package://gummi_base_template/meshes/j1_Link.STL" />
-      </geometry>
-      <material
-        name="">
-        <color
-          rgba="0.79216 0.81961 0.93333 1" />
-      </material>
-    </visual>
-    <collision>
-      <origin
-        xyz="0 0 0"
-        rpy="0 0 0" />
-      <geometry>
-        <mesh
-          filename="package://gummi_base_template/meshes/j1_Link.STL" />
+          filename="package://gummi_base_ghost/meshes/j1_Link.STL" />
+      </geometry>
+      <material
+        name="">
+        <color
+          rgba="0.79216 0.81961 0.93333 1" />
+      </material>
+    </visual>
+    <collision>
+      <origin
+        xyz="0 0 0"
+        rpy="0 0 0" />
+      <geometry>
+        <mesh
+          filename="package://gummi_base_ghost/meshes/j1_Link.STL" />
       </geometry>
     </collision>
@@ -125,19 +125,19 @@
       <geometry>
         <mesh
-          filename="package://gummi_base_template/meshes/j2_Link.STL" />
-      </geometry>
-      <material
-        name="">
-        <color
-          rgba="0.79216 0.81961 0.93333 1" />
-      </material>
-    </visual>
-    <collision>
-      <origin
-        xyz="0 0 0"
-        rpy="0 0 0" />
-      <geometry>
-        <mesh
-          filename="package://gummi_base_template/meshes/j2_Link.STL" />
+          filename="package://gummi_base_ghost/meshes/j2_Link.STL" />
+      </geometry>
+      <material
+        name="">
+        <color
+          rgba="0.79216 0.81961 0.93333 1" />
+      </material>
+    </visual>
+    <collision>
+      <origin
+        xyz="0 0 0"
+        rpy="0 0 0" />
+      <geometry>
+        <mesh
+          filename="package://gummi_base_ghost/meshes/j2_Link.STL" />
       </geometry>
     </collision>
@@ -186,19 +186,19 @@
       <geometry>
         <mesh
-          filename="package://gummi_base_template/meshes/j3_Link.STL" />
-      </geometry>
-      <material
-        name="">
-        <color
-          rgba="0.79216 0.81961 0.93333 1" />
-      </material>
-    </visual>
-    <collision>
-      <origin
-        xyz="0 0 0"
-        rpy="0 0 0" />
-      <geometry>
-        <mesh
-          filename="package://gummi_base_template/meshes/j3_Link.STL" />
+          filename="package://gummi_base_ghost/meshes/j3_Link.STL" />
+      </geometry>
+      <material
+        name="">
+        <color
+          rgba="0.79216 0.81961 0.93333 1" />
+      </material>
+    </visual>
+    <collision>
+      <origin
+        xyz="0 0 0"
+        rpy="0 0 0" />
+      <geometry>
+        <mesh
+          filename="package://gummi_base_ghost/meshes/j3_Link.STL" />
       </geometry>
     </collision>
@@ -247,19 +247,19 @@
       <geometry>
         <mesh
-          filename="package://gummi_base_template/meshes/j4_Link.STL" />
-      </geometry>
-      <material
-        name="">
-        <color
-          rgba="0.79216 0.81961 0.93333 1" />
-      </material>
-    </visual>
-    <collision>
-      <origin
-        xyz="0 0 0"
-        rpy="0 0 0" />
-      <geometry>
-        <mesh
-          filename="package://gummi_base_template/meshes/j4_Link.STL" />
+          filename="package://gummi_base_ghost/meshes/j4_Link.STL" />
+      </geometry>
+      <material
+        name="">
+        <color
+          rgba="0.79216 0.81961 0.93333 1" />
+      </material>
+    </visual>
+    <collision>
+      <origin
+        xyz="0 0 0"
+        rpy="0 0 0" />
+      <geometry>
+        <mesh
+          filename="package://gummi_base_ghost/meshes/j4_Link.STL" />
       </geometry>
     </collision>
