Commit message: finally parametrized urdf file for base

File: xacro/gummi_description_base.urdf.xacro (robot description, xacro)
@@ -23,19 +23,19 @@
       <geometry>
         <mesh
-          filename="package://gummi_base_ghost/meshes/base_link.STL" />
-      </geometry>
-      <material
-        name="">
-        <color
-          rgba="0.79216 0.81961 0.93333 1" />
-      </material>
-    </visual>
-    <collision>
-      <origin
-        xyz="0 0 0"
-        rpy="0 0 0" />
-      <geometry>
-        <mesh
-          filename="package://gummi_base_ghost/meshes/base_link.STL" />
+          filename="package://gummi_base_$(env ROS_GUMMI_BASE)/meshes/base_link.STL" />
+      </geometry>
+      <material
+        name="">
+        <color
+          rgba="0.79216 0.81961 0.93333 1" />
+      </material>
+    </visual>
+    <collision>
+      <origin
+        xyz="0 0 0"
+        rpy="0 0 0" />
+      <geometry>
+        <mesh
+          filename="package://gummi_base_$(env ROS_GUMMI_BASE)/meshes/base_link.STL" />
       </geometry>
     </collision>
@@ -64,19 +64,19 @@
       <geometry>
         <mesh
-          filename="package://gummi_base_ghost/meshes/j1_Link.STL" />
-      </geometry>
-      <material
-        name="">
-        <color
-          rgba="0.79216 0.81961 0.93333 1" />
-      </material>
-    </visual>
-    <collision>
-      <origin
-        xyz="0 0 0"
-        rpy="0 0 0" />
-      <geometry>
-        <mesh
-          filename="package://gummi_base_ghost/meshes/j1_Link.STL" />
+          filename="package://gummi_base_$(env ROS_GUMMI_BASE)/meshes/j1_Link.STL" />
+      </geometry>
+      <material
+        name="">
+        <color
+          rgba="0.79216 0.81961 0.93333 1" />
+      </material>
+    </visual>
+    <collision>
+      <origin
+        xyz="0 0 0"
+        rpy="0 0 0" />
+      <geometry>
+        <mesh
+          filename="package://gummi_base_$(env ROS_GUMMI_BASE)/meshes/j1_Link.STL" />
       </geometry>
     </collision>
@@ -125,19 +125,19 @@
       <geometry>
         <mesh
-          filename="package://gummi_base_ghost/meshes/j2_Link.STL" />
-      </geometry>
-      <material
-        name="">
-        <color
-          rgba="0.79216 0.81961 0.93333 1" />
-      </material>
-    </visual>
-    <collision>
-      <origin
-        xyz="0 0 0"
-        rpy="0 0 0" />
-      <geometry>
-        <mesh
-          filename="package://gummi_base_ghost/meshes/j2_Link.STL" />
+          filename="package://gummi_base_$(env ROS_GUMMI_BASE)/meshes/j2_Link.STL" />
+      </geometry>
+      <material
+        name="">
+        <color
+          rgba="0.79216 0.81961 0.93333 1" />
+      </material>
+    </visual>
+    <collision>
+      <origin
+        xyz="0 0 0"
+        rpy="0 0 0" />
+      <geometry>
+        <mesh
+          filename="package://gummi_base_$(env ROS_GUMMI_BASE)/meshes/j2_Link.STL" />
       </geometry>
     </collision>
@@ -186,19 +186,19 @@
       <geometry>
         <mesh
-          filename="package://gummi_base_ghost/meshes/j3_Link.STL" />
-      </geometry>
-      <material
-        name="">
-        <color
-          rgba="0.79216 0.81961 0.93333 1" />
-      </material>
-    </visual>
-    <collision>
-      <origin
-        xyz="0 0 0"
-        rpy="0 0 0" />
-      <geometry>
-        <mesh
-          filename="package://gummi_base_ghost/meshes/j3_Link.STL" />
+          filename="package://gummi_base_$(env ROS_GUMMI_BASE)/meshes/j3_Link.STL" />
+      </geometry>
+      <material
+        name="">
+        <color
+          rgba="0.79216 0.81961 0.93333 1" />
+      </material>
+    </visual>
+    <collision>
+      <origin
+        xyz="0 0 0"
+        rpy="0 0 0" />
+      <geometry>
+        <mesh
+          filename="package://gummi_base_$(env ROS_GUMMI_BASE)/meshes/j3_Link.STL" />
       </geometry>
     </collision>
@@ -247,19 +247,19 @@
       <geometry>
         <mesh
-          filename="package://gummi_base_ghost/meshes/j4_Link.STL" />
-      </geometry>
-      <material
-        name="">
-        <color
-          rgba="0.79216 0.81961 0.93333 1" />
-      </material>
-    </visual>
-    <collision>
-      <origin
-        xyz="0 0 0"
-        rpy="0 0 0" />
-      <geometry>
-        <mesh
-          filename="package://gummi_base_ghost/meshes/j4_Link.STL" />
+          filename="package://gummi_base_$(env ROS_GUMMI_BASE)/meshes/j4_Link.STL" />
+      </geometry>
+      <material
+        name="">
+        <color
+          rgba="0.79216 0.81961 0.93333 1" />
+      </material>
+    </visual>
+    <collision>
+      <origin
+        xyz="0 0 0"
+        rpy="0 0 0" />
+      <geometry>
+        <mesh
+          filename="package://gummi_base_$(env ROS_GUMMI_BASE)/meshes/j4_Link.STL" />
       </geometry>
     </collision>

Commit message: Tuned ghost limits and speeds.

File: xacro/gummi_description_base.urdf.xacro (robot description, xacro)
@@ -100,5 +100,5 @@
       effort="0"
       velocity="0" /> -->
-    <limit effort="0" lower="-0.52" upper="1.04" velocity="1.0"/>
+    <limit effort="0" lower="-0.79" upper="1.04" velocity="1.0"/>
   </joint>
   <!-- j2_Link -->
@@ -161,5 +161,5 @@
       effort="0"
       velocity="0" /> -->
-    <limit effort="0" lower="-0.55" upper="1.4" velocity="1.0"/>
+    <limit effort="0" lower="-0.95" upper="2.3" velocity="1.0"/>
   </joint>
   <!-- j3_Link -->

Commit message: Ok on ghost.

File: xacro/gummi_description_base.urdf.xacro (robot description, xacro)
@@ -100,5 +100,5 @@
       effort="0"
       velocity="0" /> -->
-    <limit effort="0" lower="-0.79" upper="1.04" velocity="1.0"/>
+    <limit effort="0" lower="-0.75" upper="1.0" velocity="1.0"/>
   </joint>
   <!-- j2_Link -->
@@ -283,5 +283,5 @@
       effort="0"
       velocity="0" /> -->
-    <limit effort="0" lower="-1.57080" upper="1.57080" velocity="1.0"/>
+    <limit effort="0" lower="-1.56" upper="1.56" velocity="1.0"/>
   </joint>
 </robot>
