Commit message: Important commit: made fastswitch into default. Removed unused stl files.

File: xacro/gummi_base.srdf.xacro (robot description, xacro)
@@ -34,13 +34,13 @@
 <xacro:macro name="disable_collisions_mixed">
   <!--MIXED DISABLE COLLISIONS FOR BASE EE COLISIONS: set by hand or remove! -->
-  <disable_collisions link1="base_link" link2="lowerarm_preroll" reason="Never" />
+  <disable_collisions link1="base_link" link2="lowerarm_preroll_u" reason="Never" />
   <disable_collisions link1="lowerarm" link2="shoulder" reason="Never" />
   <disable_collisions link1="lowerarm" link2="shoulder_preroll" reason="Never" />
   <disable_collisions link1="lowerarm" link2="upperarm" reason="Never" />
   <disable_collisions link1="lowerarm" link2="upperarm_preroll" reason="Never" />
-  <disable_collisions link1="lowerarm_preroll" link2="shoulder" reason="Never" />
-  <disable_collisions link1="lowerarm_preroll" link2="shoulder_preroll" reason="Never" />
-  <disable_collisions link1="lowerarm_preroll" link2="upperarm" reason="Adjacent" />
-  <disable_collisions link1="lowerarm_preroll" link2="upperarm_preroll" reason="Never" />
+  <disable_collisions link1="lowerarm_preroll_u" link2="shoulder" reason="Never" />
+  <disable_collisions link1="lowerarm_preroll_u" link2="shoulder_preroll" reason="Never" />
+  <disable_collisions link1="lowerarm_preroll_u" link2="upperarm" reason="Adjacent" />
+  <disable_collisions link1="lowerarm_preroll_u" link2="upperarm_preroll" reason="Never" />
 </xacro:macro>
 </robot>

File: xacro/gummi_description_base.urdf.xacro (robot description, xacro)
@@ -285,3 +285,62 @@
     <limit effort="0" lower="-1.56" upper="1.56" velocity="1.0"/>
   </joint>
+  <!-- j5_Link -->
+<link
+  name="lowerarm_preroll_u">
+  <inertial>
+    <origin
+      xyz="0.0480680914336555 -0.0154122894983864 -0.00982448117120333"
+      rpy="0 0 0" />
+    <mass
+      value="0.0573776116734678" />
+    <inertia
+      ixx="1.98794332161084E-05"
+      ixy="-1.22203388710061E-06"
+      ixz="5.63209252093047E-06"
+      iyy="4.47548061016055E-05"
+      iyz="2.39819214170021E-07"
+      izz="4.43764478788868E-05" />
+  </inertial>
+  <visual>
+    <origin
+      xyz="0 0 0"
+      rpy="0 0 0" />
+    <geometry>
+      <mesh
+        filename="package://gummi_base_$(env ROS_GUMMI_BASE)/meshes/j5_Link.STL" />
+    </geometry>
+    <material name="">
+      <color rgba="1 0.7 0.7 1"/>
+    </material>
+  </visual>
+  <collision>
+    <origin
+      xyz="0 0 0"
+      rpy="0 0 0" />
+    <geometry>
+      <mesh
+        filename="package://gummi_base_$(env ROS_GUMMI_BASE)/meshes/j5_Link.STL" />
+    </geometry>
+  </collision>
+</link>
+<!-- j5 -->
+<joint
+  name="elbow"
+  type="revolute">
+  <origin
+    xyz="0 0.01475 -0.19105"
+    rpy="0 0 0" />
+  <parent
+    link="upperarm" />
+  <child
+    link="lowerarm_preroll_u" />
+  <axis
+    xyz="0 -1 0" />
+  <!-- <limit
+    lower="-1.5708"
+    upper="1.5708"
+    effort="0"
+    velocity="0" /> -->
+  <limit effort="0" lower="-0.72" upper="0.32" velocity="1.0"/>
+</joint>
 </robot>

Commit message: making changes to use new dovetail design

File: xacro/gummi_base.srdf.xacro (robot description, xacro)
@@ -8,4 +8,6 @@
   <joint name="shoulder_pitch" />
   <joint name="upperarm_roll" />
+  <joint name="elbow" />
+  <joint name="fastswitch" />
 </xacro:macro>
 <xacro:macro name="group_state_right_arm_base">
@@ -14,4 +16,5 @@
   <joint name="shoulder_yaw" value="0" />
   <joint name="upperarm_roll" value="0" />
+  <joint name="elbow" value="0" />
 </xacro:macro>
 <xacro:macro name="virtual_joints_base">
@@ -43,4 +46,5 @@
   <disable_collisions link1="lowerarm_preroll_u" link2="upperarm" reason="Adjacent" />
   <disable_collisions link1="lowerarm_preroll_u" link2="upperarm_preroll" reason="Never" />
+  <disable_collisions link1="lowerarm_preroll_u" link2="lowerarm_preroll_d" reason="Adjacent" />
 </xacro:macro>
 </robot>

File: xacro/gummi_description_base.urdf.xacro (robot description, xacro)
@@ -5,15 +5,15 @@
     <inertial>
       <origin
-        xyz="-0.096576 0.093216 -0.5062"
-        rpy="0 0 0" />
-      <mass
-        value="6.6524" />
-      <inertia
-        ixx="1.072"
-        ixy="0.0014296"
-        ixz="-0.066318"
-        iyy="1.1363"
-        iyz="0.0042533"
-        izz="0.20948" />
+        xyz="-9.81410393552373E-06 -0.0460000689343235 -0.0065295158451983"
+        rpy="0 0 0" />
+      <mass
+        value="0.335467320988356" />
+      <inertia
+        ixx="4.37751934245478E-05"
+        ixy="-7.25114187919924E-08"
+        ixz="-1.8551473383786E-07"
+        iyy="3.79746167195594E-05"
+        iyz="-1.48426357415501E-05"
+        izz="5.80238931250525E-06" />
     </inertial>
     <visual>
@@ -28,5 +28,5 @@
         name="">
         <color
-          rgba="0.79216 0.81961 0.93333 1" />
+          rgba="0.792156862745098 0.819607843137255 0.933333333333333 1" />
       </material>
     </visual>
@@ -41,51 +41,49 @@
     </collision>
   </link>
-  <!-- j1_Link -->
   <link
     name="shoulder_preroll">
     <inertial>
       <origin
-        xyz="-3.1428E-06 -0.0073636 0.053528"
-        rpy="0 0 0" />
-      <mass
-        value="0.42246" />
-      <inertia
-        ixx="0.0013384"
-        ixy="6.4017E-08"
-        ixz="6.2475E-08"
-        iyy="0.0012663"
-        iyz="0.00011953"
-        izz="0.00092802" />
-    </inertial>
-    <visual>
-      <origin
-        xyz="0 0 0"
-        rpy="0 0 0" />
-      <geometry>
-        <mesh
-          filename="package://gummi_base_$(env ROS_GUMMI_BASE)/meshes/j1_Link.STL" />
-      </geometry>
-      <material
-        name="">
-        <color
-          rgba="0.79216 0.81961 0.93333 1" />
-      </material>
-    </visual>
-    <collision>
-      <origin
-        xyz="0 0 0"
-        rpy="0 0 0" />
-      <geometry>
-        <mesh
-          filename="package://gummi_base_$(env ROS_GUMMI_BASE)/meshes/j1_Link.STL" />
-      </geometry>
-    </collision>
-  </link>
-  <!-- j1 -->
+        xyz="-2.1762E-05 -0.0041376 0.031717"
+        rpy="0 0 0" />
+      <mass
+        value="0.77225" />
+      <inertia
+        ixx="0.0026527"
+        ixy="1.2427E-07"
+        ixz="5.0677E-07"
+        iyy="0.003032"
+        iyz="4.4108E-05"
+        izz="0.0012294" />
+    </inertial>
+    <visual>
+      <origin
+        xyz="0 0 0"
+        rpy="0 0 0" />
+      <geometry>
+        <mesh
+          filename="package://gummi_base_$(env ROS_GUMMI_BASE)/meshes/shoulder_preroll.STL" />
+      </geometry>
+      <material
+        name="">
+        <color
+          rgba="0.79216 0.81961 0.93333 1" />
+      </material>
+    </visual>
+    <collision>
+      <origin
+        xyz="0 0 0"
+        rpy="0 0 0" />
+      <geometry>
+        <mesh
+          filename="package://gummi_base_$(env ROS_GUMMI_BASE)/meshes/shoulder_preroll.STL" />
+      </geometry>
+    </collision>
+  </link>
   <joint
     name="shoulder_yaw"
     type="revolute">
     <origin
-      xyz="0 0 0"
+      xyz="-0.00027025 -0.10997 0.008"
       rpy="0 0 0" />
     <parent
@@ -94,59 +92,56 @@
       link="shoulder_preroll" />
     <axis
-      xyz="0 0 1" />
-    <!-- <limit
-      lower="-1.5708"
-      upper="1.5708"
+      xyz="0 0 -1" />
+    <limit
+      lower="-0.75"
+      upper="1"
       effort="0"
-      velocity="0" /> -->
-    <limit effort="0" lower="-0.75" upper="1.0" velocity="1.0"/>
-  </joint>
-  <!-- j2_Link -->
+      velocity="0" />
+  </joint>
   <link
     name="shoulder">
     <inertial>
       <origin
-        xyz="-7.4885E-05 -0.045317 5.3695E-06"
-        rpy="0 0 0" />
-      <mass
-        value="0.29147" />
-      <inertia
-        ixx="0.00040953"
-        ixy="-1.1184E-06"
-        ixz="-1.4753E-06"
-        iyy="0.00026628"
-        iyz="5.6545E-08"
-        izz="0.00048004" />
-    </inertial>
-    <visual>
-      <origin
-        xyz="0 0 0"
-        rpy="0 0 0" />
-      <geometry>
-        <mesh
-          filename="package://gummi_base_$(env ROS_GUMMI_BASE)/meshes/j2_Link.STL" />
-      </geometry>
-      <material
-        name="">
-        <color
-          rgba="0.79216 0.81961 0.93333 1" />
-      </material>
-    </visual>
-    <collision>
-      <origin
-        xyz="0 0 0"
-        rpy="0 0 0" />
-      <geometry>
-        <mesh
-          filename="package://gummi_base_$(env ROS_GUMMI_BASE)/meshes/j2_Link.STL" />
-      </geometry>
-    </collision>
-  </link>
-  <!-- j2 -->
+        xyz="-6.6912E-05 -0.10412 4.2145E-06"
+        rpy="0 0 0" />
+      <mass
+        value="0.32611" />
+      <inertia
+        ixx="0.00024984"
+        ixy="-1.3E-06"
+        ixz="1.74E-07"
+        iyy="7.3364E-05"
+        iyz="8.2134E-08"
+        izz="0.0003232" />
+    </inertial>
+    <visual>
+      <origin
+        xyz="0 0 0"
+        rpy="0 0 0" />
+      <geometry>
+        <mesh
+          filename="package://gummi_base_$(env ROS_GUMMI_BASE)/meshes/shoulder.STL" />
+      </geometry>
+      <material
+        name="">
+        <color
+          rgba="0.79216 0.81961 0.93333 1" />
+      </material>
+    </visual>
+    <collision>
+      <origin
+        xyz="0 0 0"
+        rpy="0 0 0" />
+      <geometry>
+        <mesh
+          filename="package://gummi_base_$(env ROS_GUMMI_BASE)/meshes/shoulder.STL" />
+      </geometry>
+    </collision>
+  </link>
   <joint
     name="shoulder_roll"
     type="revolute">
     <origin
-      xyz="0 0 0.126"
+      xyz="-2.6378E-05 0.057605 0.1302"
       rpy="0 0 0" />
     <parent
@@ -155,59 +150,56 @@
       link="shoulder" />
     <axis
-      xyz="0 -1 0" />
-    <!-- <limit
-      lower="-1.5708"
-      upper="1.5708"
+      xyz="0 1 0" />
+    <limit
+      lower="-0.95"
+      upper="2.3"
       effort="0"
-      velocity="0" /> -->
-    <limit effort="0" lower="-0.95" upper="2.3" velocity="1.0"/>
-  </joint>
-  <!-- j3_Link -->
+      velocity="0" />
+  </joint>
   <link
     name="upperarm_preroll">
     <inertial>
       <origin
-        xyz="-0.0021446 -0.0092567 -0.047728"
-        rpy="0 0 0" />
-      <mass
-        value="0.10451" />
-      <inertia
-        ixx="5.4001E-05"
-        ixy="5.1914E-07"
-        ixz="-6.0861E-06"
-        iyy="7.317E-05"
-        iyz="-6.031E-07"
-        izz="4.6633E-05" />
-    </inertial>
-    <visual>
-      <origin
-        xyz="0 0 0"
-        rpy="0 0 0" />
-      <geometry>
-        <mesh
-          filename="package://gummi_base_$(env ROS_GUMMI_BASE)/meshes/j3_Link.STL" />
-      </geometry>
-      <material
-        name="">
-        <color
-          rgba="0.79216 0.81961 0.93333 1" />
-      </material>
-    </visual>
-    <collision>
-      <origin
-        xyz="0 0 0"
-        rpy="0 0 0" />
-      <geometry>
-        <mesh
-          filename="package://gummi_base_$(env ROS_GUMMI_BASE)/meshes/j3_Link.STL" />
-      </geometry>
-    </collision>
-  </link>
-  <!-- j3 -->
+        xyz="0.031774 -0.0098005 -0.046115"
+        rpy="0 0 0" />
+      <mass
+        value="0.11889" />
+      <inertia
+        ixx="4.0724E-05"
+        ixy="7.0589E-07"
+        ixz="1.4611E-05"
+        iyy="6.3279E-05"
+        iyz="6.4487E-07"
+        izz="2.3476E-05" />
+    </inertial>
+    <visual>
+      <origin
+        xyz="0 0 0"
+        rpy="0 0 0" />
+      <geometry>
+        <mesh
+          filename="package://gummi_base_$(env ROS_GUMMI_BASE)/meshes/upperarm_preroll.STL" />
+      </geometry>
+      <material
+        name="">
+        <color
+          rgba="0.79216 0.81961 0.93333 1" />
+      </material>
+    </visual>
+    <collision>
+      <origin
+        xyz="0 0 0"
+        rpy="0 0 0" />
+      <geometry>
+        <mesh
+          filename="package://gummi_base_$(env ROS_GUMMI_BASE)/meshes/upperarm_preroll.STL" />
+      </geometry>
+    </collision>
+  </link>
   <joint
     name="shoulder_pitch"
     type="revolute">
     <origin
-      xyz="0 -0.1185 0"
+      xyz="-0.024 -0.17679 8.6827E-05"
       rpy="0 0 0" />
     <parent
@@ -217,58 +209,55 @@
     <axis
       xyz="-1 0 0" />
-<!-- <limit
-      lower="-1.5708"
-      upper="1.5708"
+    <limit
+      lower="-0.15"
+      upper="1.1"
       effort="0"
-      velocity="0" /> -->
-    <limit effort="0" lower="-0.15" upper="1.1" velocity="1.0"/>
-  </joint>
-  <!-- j4_Link -->
+      velocity="0" />
+  </joint>
   <link
     name="upperarm">
     <inertial>
       <origin
-        xyz="-0.0024868 -9.272E-05 -0.088372"
-        rpy="0 0 0" />
-      <mass
-        value="0.23537" />
-      <inertia
-        ixx="0.00067545"
-        ixy="5.6472E-08"
-        ixz="1.0957E-05"
-        iyy="0.00067994"
-        iyz="-1.7347E-06"
-        izz="6.6647E-05" />
-    </inertial>
-    <visual>
-      <origin
-        xyz="0 0 0"
-        rpy="0 0 0" />
-      <geometry>
-        <mesh
-          filename="package://gummi_base_$(env ROS_GUMMI_BASE)/meshes/j4_Link.STL" />
-      </geometry>
-      <material
-        name="">
-        <color
-          rgba="0.79216 0.81961 0.93333 1" />
-      </material>
-    </visual>
-    <collision>
-      <origin
-        xyz="0 0 0"
-        rpy="0 0 0" />
-      <geometry>
-        <mesh
-          filename="package://gummi_base_$(env ROS_GUMMI_BASE)/meshes/j4_Link.STL" />
-      </geometry>
-    </collision>
-  </link>
-  <!-- j4 -->
+        xyz="-0.0024737 -8.3239E-05 -0.1319"
+        rpy="0 0 0" />
+      <mass
+        value="0.26501" />
+      <inertia
+        ixx="0.00079812"
+        ixy="-7.2143E-08"
+        ixz="-4.087E-05"
+        iyy="0.0007849"
+        iyz="-1.9447E-06"
+        izz="2.1965E-05" />
+    </inertial>
+    <visual>
+      <origin
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